File: hardware/KungFuFlash2.kicad_pcb (KiCad board)
At the start: 2 copper layers, 60.6 x 62 mm, 53 parts, among them J1 SWD, J2 USB_B_Micro, J3 Wifi, Q1 BC817, SW1 Reset, SW2 Menu, SW3 Special, U1 C64-Exp-Port, U2 AMS1117-3.3, U3 STM32H7B0VBTx, Y1 25MHz

Commit message: Add USB C and JLCPCB files
Parts:
- removed J2: USB_B_Micro, KungFuFlash2:Conn_USBmicro-B_ebay-side_TH
- added J4: USB_C_Receptacle_USB2.0, Connector_USB:USB_C_Receptacle_XKB_U262-16XN-4BVC11, F.Cu at (132.7, 86.5)
- added R16: 10k, Resistor_SMD:R_0805_2012Metric_Pad1.20x1.40mm_HandSolder, F.Cu at (131.7, 80.0)
- added R17: 10k, Resistor_SMD:R_0805_2012Metric_Pad1.20x1.40mm_HandSolder, F.Cu at (131.8, 92.8)
- Y1: value 25MHz -> 25 MHz; footprint Crystal:Crystal_SMD_5032-2Pin_5.0x3.2mm -> Crystal:Crystal_SMD_3225-4Pin_3.2x2.5mm
- moved D3 1.29 mm to (126.1, 85.1)
- moved Y1 0.21 mm to (96.0, 102.4), turned to 90 degrees
Connections:
- Y1 pad 1: Net-(U3-PH0) -> Net-(U3-PH1)
- Y1 pad 2: Net-(U3-PH1) -> GND
Routing:
- net GND: track 705.4 -> 660.5 mm, vias 77 -> 78
- net /USB_DP: track 23.0 -> 31.8 mm, vias 0 -> 2
- net Net-(J4-CC1): track 0.00 -> 8.63 mm
- net Net-(J4-CC2): track 0.00 -> 7.28 mm
- net /USB_DM: track 22.9 -> 27.9 mm, vias 0 -> 2
- net Net-(U3-PH0): track 8.27 -> 10.3 mm
- net +3V3: track 276.9 -> 275.6 mm
- net Net-(U3-PH1): track 8.44 -> 7.61 mm
- net +5C: track 7.91 -> 8.62 mm, vias 2 -> 0
- net Net-(D2-K): track 81.4 -> 80.8 mm

Commit message: Update PCB for USBC resistors 5.1k and production files
Parts:
- R16, R17: value 10k -> 5.1k
Changed lines of the file:
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@@
         (effects (font (size 1 1) (thickness 0.15)))
     )
-    (fp_text value "10k" (at 0 1.65) (layer "F.Fab")
+    (fp_text value "5.1k" (at 0 1.65) (layer "F.Fab")
         (effects (font (size 1 1) (thickness 0.15)))
     )
@@
         (effects (font (size 1 1) (thickness 0.15)))
     )
-    (fp_text value "10k" (at 0 1.65) (layer "F.Fab")
+    (fp_text value "5.1k" (at 0 1.65) (layer "F.Fab")
         (effects (font (size 1 1) (thickness 0.15)))
     )

Commit message: SMT buttons
Parts:
- added REF**: WEEE-Logo_5.6x8mm_SilkScreen, Symbol:WEEE-Logo_5.6x8mm_SilkScreen, B.Cu at (80.9, 74.5)
- added REF**: CE-Logo_8.5x6mm_SilkScreen, Symbol:CE-Logo_8.5x6mm_SilkScreen, B.Cu at (90.5, 74.7)
- SW1, SW2, SW3: footprint Button_Switch_THT:SW_PUSH_6mm_H8mm -> Button_Switch_SMD:SW_SPST_PTS645
- moved SW1 4.01 mm to (127.0, 72.6)
- moved SW2 3.96 mm to (115.6, 72.6)
- moved SW3 3.90 mm to (82.8, 72.6)
Routing:
- net /~{RST}: track 56.2 -> 60.1 mm, vias 4 -> 6
- net Net-(R5-Pad1): track 8.77 -> 10.2 mm
- net GND: track 660.5 -> 659.7 mm
Other:
- board text added: "Kung Fu Flash 2"
- board text removed: "locked"
